Commit message: 3finger gripper added

File: description/arm.xacro (robot description, xacro)
@@ -3,11 +3,11 @@
   <!-- include macro definitions -->
   <xacro:include filename="$(find ur_description)/urdf/inc/ur5e_macro.xacro"/>
-  <xacro:ur5e_robot prefix="ur5e_"/>
+  <xacro:ur5e_robot prefix=""/>
   <xacro:include filename="$(find robotiq_3f_gripper_visualization)/cfg/robotiq-3f-gripper_articulated_macro.xacro"/>
-  <xacro:robotiq-3f-gripper_articulated prefix="s_model_"/>
+  <xacro:robotiq-3f-gripper_articulated prefix="gripper_"/>
     <!-- attach eef to ur5 model -->
     <joint name="gripper_joint" type="fixed">
-      <parent link="ur5e_wrist_3_link" />
-      <child link = "s_model_palm" />
+      <parent link="wrist_3_link" />
+      <child link = "gripper_palm" />
       <origin xyz="0.0 0.0 0.057" rpy="${pi/2} 0.0 0.0" />
     </joint>

Commit message: setup gripper moveit config

File: description/arm.xacro (robot description, xacro)
@@ -8,5 +8,5 @@
     <!-- attach eef to ur5 model -->
     <joint name="gripper_joint" type="fixed">
-      <parent link="wrist_3_link" />
+      <parent link="tool0" />
       <child link = "gripper_palm" />
       <origin xyz="0.0 0.0 0.057" rpy="${pi/2} 0.0 0.0" />

Commit message: corrected the arm.xacro file and redid the setup using Moveit

File: description/arm.xacro (robot description, xacro)
@@ -1,10 +1,13 @@
 <?xml version="1.0"?>
-<robot xmlns:xacro="http://www.ros.org/wiki/xacro" name="arm" >
+<robot xmlns:xacro="http://www.ros.org/wiki/xacro" name="ur_robot_with_gripper" >
   <!-- include macro definitions -->
   <xacro:include filename="$(find ur_description)/urdf/inc/ur5e_macro.xacro"/>
+  <xacro:include filename="$(find robotiq_3f_gripper_visualization)/cfg/robotiq-3f-gripper_articulated_macro.xacro"/>
+  <!-- Create a new macro to link both -->
+  <xacro:macro name="ur_robotiq" params="prefix">
+  <!-- instantiate both -->
   <xacro:ur5e_robot prefix=""/>
-  <xacro:include filename="$(find robotiq_3f_gripper_visualization)/cfg/robotiq-3f-gripper_articulated_macro.xacro"/>
   <xacro:robotiq-3f-gripper_articulated prefix="gripper_"/>
-    <!-- attach eef to ur5 model -->
+  <!-- attach griper to ur5 model -->
     <joint name="gripper_joint" type="fixed">
       <parent link="tool0" />
@@ -12,3 +15,6 @@
       <origin xyz="0.0 0.0 0.057" rpy="${pi/2} 0.0 0.0" />
     </joint>
+  </xacro:macro>
+  <!-- Now instantiate above macro -->
+ <xacro:ur_robotiq prefix=""/>
 </robot>
