Commit message: tracking tags is now working, motion planning needs to be made optimal

File: description/workcell.xacro (robot description, xacro)
@@ -24,5 +24,5 @@
     <collision>
       <geometry>
-        <box size="2.0 2.0 0.05"/>
+        <box size="2.0 2.0 0.1"/>
       </geometry>
     </collision>
